File: Board/STM32GenericBoard/STM32GenericBoard.kicad_pcb (KiCad board)
At the start: 6 copper layers, 50.8 x 50.8 mm, 63 parts, among them J1 USB_B_Micro, J2 Conn_01x08_Pin, U1 STM32H743VGTx, U2 AMS1117-3.3, U3 ICM-45686, Y1 Crystal_GND24

Commit message: save
Parts:
- removed R1, R2: 10k, Resistor_SMD:R_0402_1005Metric_Pad0.72x0.64mm_HandSolder
- added C17: 100n, Capacitor_SMD:C_0402_1005Metric_Pad0.74x0.62mm_HandSolder, F.Cu at (100.9, 48.1)
- UCAN1, UCAN2: value SN65HVD230 -> SN65HVD234
- moved C6 1.79 mm to (99.9, 45.3)
- moved C18 0.57 mm to (98.5, 48.3)
- moved J1 0.54 mm to (137.9, 36.9)
- renumbered PWR+5V1 to +5V1, Encoder1 to Encoder1/T2, Encoder2 to Encoder2/T4
Connections:
- UCAN1 pad 8: Net-(UCAN1-Rs) -> +3V3
- UCAN2 pad 8: Net-(UCAN2-Rs) -> +3V3
Routing:
- net Net-(UCAN1-Rs): track 8.00 -> 0.00 mm, vias 2 -> 0
- net GND: track 72.9 -> 79.1 mm, vias 42 -> 41
- net +3V3: track 51.1 -> 56.1 mm, vias 31 -> 33
- net Net-(UCAN2-Rs): track 1.91 -> 0.00 mm
- net FDCAN2_TX: track 24.9 -> 26.5 mm, vias 1 -> 2
- net USB_OTG_P: track 26.3 -> 27.2 mm
- net FDCAN1_RX: track 25.2 -> 26.0 mm
- net PE5_SPI2_CS: track 30.7 -> 31.4 mm
- net USB_OTG_N: track 29.6 -> 30.2 mm
- net UART4_TX: vias 3 -> 2
- net PE6_SPI3_CS: vias 1 -> 2
- net NRST: vias 4 -> 3
Other:
- board text added: "E4 MO MI SC + G"
- board text added: "E5 MO MI SC + G"
- board text added: "E8 E7 B2 B1 B0 C5 + G"
- board text added: "G"
- board text added: "L H"
- board text added: "RX TX + G"
- board text added: "TIM1"
- board text added: "U7 RST IO CK + G"
- board text added: "Z C1 C2 + G"
