File: Board/STM32GenericBoard/STM32GenericBoard.kicad_sch (KiCad schematic)
At the start: 39 parts, among them U1 STM32H743VGTx, U2 AMS1117-3.3, U3 ICM-45686, Y1 Crystal_GND24

Commit message: feat(telemetry): add WiFi UDP bridge and UART4 DMA streaming
Add ESP32 bridge, TelemetryServer, and STM32 BalanceFrame at 200 Hz/921600.

Fix UART4 TC IRQ for HAL DMA TX completion, RPC gain tuning, and NVIC setup.

Co-authored-by: Cursor <cursoragent@cursor.com>
Connections:
- net +3V3: now also UCAN1.5 (Vref), UCAN2.5 (Vref); no longer UCAN1.8 (Rs), UCAN2.8 (Rs)
- net GND: now also UCAN1.8 (Rs), UCAN2.8 (Rs)
- no-connect marks 44 -> 42
Changed lines of the file:
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@@
 	)
 	(no_connect
-		(at 121.92 116.84)
-	)
-	(no_connect
 		(at 33.02 128.27)
 	)
@@
 	)
 	(no_connect
-		(at 121.92 138.43)
-	)
-	(no_connect
 		(at 182.88 96.52)
 	)
@@
 	(wire
 		(pts
-			(xy 114.3 140.97) (xy 121.92 140.97)
-		)
-		(stroke
-			(width 0)
-			(type default)
-		)
-	)
-	(wire
-		(pts
 			(xy 33.02 179.07) (xy 30.48 179.07)
 		)
@@
 	(wire
 		(pts
-			(xy 114.3 119.38) (xy 121.92 119.38)
-		)
-		(stroke
-			(width 0)
-			(type default)
-		)
-	)
-	(wire
-		(pts
 			(xy 34.29 20.32) (xy 39.37 20.32)
 		)
@@
 	)
 	(symbol
+		(lib_id "power:GND")
+		(at 121.92 140.97 270)
+		(unit 1)
+		(body_style 1)
+		(exclude_from_sim no)
+		(in_bom yes)
+		(on_board yes)
+		(in_pos_files yes)
+		(dnp no)
+		(property "Reference" "#PWR061"
+			(at 115.57 140.97 0)
+			(hide yes)
+			(show_name no)
+			(do_not_autoplace no)
+			(effects
+				(font
+					(size 1.27 1.27)
+				)
+			)
+		)
+		(property "Value" "GND"
+			(at 118.11 140.9701 90)
+			(show_name no)
+			(do_not_autoplace no)
+			(effects
+				(font
+					(size 1.27 1.27)
+				)
+				(justify right)
+			)
+		)
+		(property "Footprint" ""
+			(at 121.92 140.97 0)
+			(hide yes)
+			(show_name no)
+			(do_not_autoplace no)
+			(effects
+				(font
+					(size 1.27 1.27)
+				)
+			)
+		)
+		(property "Datasheet" ""
+			(at 121.92 140.97 0)
+			(hide yes)
+			(show_name no)
+			(do_not_autoplace no)
+			(effects
+				(font
+					(size 1.27 1.27)
+				)
+			)
+		)
+		(property "Description" "Power symbol creates a global label with name \"GND\" , ground"
+			(at 121.92 140.97 0)
+			(hide yes)
+			(show_name no)
+			(do_not_autoplace no)
+			(effects
+				(font
+					(size 1.27 1.27)
+				)
+			)
+		)
+		(pin "1"
+		)
+		(instances
+			(project "STM32GenericBoard"
+				(path "/55bb8da0-81e5-46ef-8fd3-f4a6b9d14d56"
+					(reference "#PWR061")
+					(unit 1)
+				)
+			)
+		)
+	)
+	(symbol
 		(lib_id "Device:C")
 		(at 54.61 24.13 0)
@@
 	(symbol
 		(lib_id "power:+3V3")
-		(at 114.3 119.38 90)
+		(at 121.92 116.84 90)
 		(unit 1)
 		(body_style 1)
@@
 		(fields_autoplaced yes)
 		(property "Reference" "#PWR059"
-			(at 118.11 119.38 0)
+			(at 125.73 116.84 0)
 			(hide yes)
 			(show_name no)
@@
 		)
 		(property "Value" "+3V3"
-			(at 110.49 119.3799 90)
+			(at 118.11 116.8399 90)
 			(show_name no)
 			(do_not_autoplace no)
@@
 		)
 		(property "Footprint" ""
-			(at 114.3 119.38 0)
+			(at 121.92 116.84 0)
 			(hide yes)
 			(show_name no)
@@
 		)
 		(property "Datasheet" ""
-			(at 114.3 119.38 0)
+			(at 121.92 116.84 0)
 			(hide yes)
 			(show_name no)
@@
 		)
 		(property "Description" "Power symbol creates a global label with name \"+3V3\""
-			(at 114.3 119.38 0)
+			(at 121.92 116.84 0)
 			(hide yes)
 			(show_name no)
@@
 	)
 	(symbol
+		(lib_id "power:GND")
+		(at 121.92 119.38 270)
+		(unit 1)
+		(body_style 1)
+		(exclude_from_sim no)
+		(in_bom yes)
+		(on_board yes)
+		(in_pos_files yes)
+		(dnp no)
+		(property "Reference" "#PWR062"
+			(at 115.57 119.38 0)
+			(hide yes)
+			(show_name no)
+			(do_not_autoplace no)
+			(effects
+				(font
+					(size 1.27 1.27)
+				)
+			)
+		)
+		(property "Value" "GND"
+			(at 118.11 119.3801 90)
+			(show_name no)
+			(do_not_autoplace no)
+			(effects
+				(font
+					(size 1.27 1.27)
+				)
+				(justify right)
+			)
+		)
+		(property "Footprint" ""
+			(at 121.92 119.38 0)
+			(hide yes)
+			(show_name no)
+			(do_not_autoplace no)
+			(effects
+				(font
+					(size 1.27 1.27)
+				)
+			)
+		)
+		(property "Datasheet" ""
+			(at 121.92 119.38 0)
+			(hide yes)
+			(show_name no)
+			(do_not_autoplace no)
+			(effects
+				(font
+					(size 1.27 1.27)
+				)
+			)
+		)
+		(property "Description" "Power symbol creates a global label with name \"GND\" , ground"
+			(at 121.92 119.38 0)
+			(hide yes)
+			(show_name no)
+			(do_not_autoplace no)
+			(effects
+				(font
+					(size 1.27 1.27)
+				)
+			)
+		)
+		(pin "1"
+		)
+		(instances
+			(project "STM32GenericBoard"
+				(path "/55bb8da0-81e5-46ef-8fd3-f4a6b9d14d56"
+					(reference "#PWR062")
+					(unit 1)
+				)
+			)
+		)
+	)
+	(symbol
 		(lib_id "power:+3V3")
-		(at 114.3 140.97 90)
+		(at 121.92 138.43 90)
 		(unit 1)
 		(body_style 1)
@@
 		(fields_autoplaced yes)
 		(property "Reference" "#PWR060"
-			(at 118.11 140.97 0)
+			(at 125.73 138.43 0)
 			(hide yes)
 			(show_name no)
@@
 		)
 		(property "Value" "+3V3"
-			(at 110.49 140.9699 90)
+			(at 118.11 138.4299 90)
 			(show_name no)
 			(do_not_autoplace no)
@@
 		)
 		(property "Footprint" ""
-			(at 114.3 140.97 0)
+			(at 121.92 138.43 0)
 			(hide yes)
 			(show_name no)
@@
 		)
 		(property "Datasheet" ""
-			(at 114.3 140.97 0)
+			(at 121.92 138.43 0)
 			(hide yes)
 			(show_name no)
@@
 		)
 		(property "Description" "Power symbol creates a global label with name \"+3V3\""
-			(at 114.3 140.97 0)
+			(at 121.92 138.43 0)
 			(hide yes)
 			(show_name no)
